Commit message: amend xacro w/ inertial macro, etc.

File: chefbot/chefbot_description/urdf/a.urdf (robot description, URDF)
Before this commit: robot turtlebot, 17 links, 16 joints
Links:
- link cliff_sensor_front_link: mass 0.0001 -> 0.01
- link cliff_sensor_left_link: mass 0.0001 -> 0.01
- link cliff_sensor_right_link: mass 0.0001 -> 0.01
- link gyro_link: mass 0.001 -> 0.01

File: chefbot/chefbot_description/urdf/chefbot_properties.urdf.xacro (robot description, xacro)
@@ -1,4 +1,5 @@
-<?xml version="1.0" encoding="utf-8"?>
-<!--
+<?xml version="1.0"?>
+<robot xmlns:xacro="http://ros.org/wiki/xacro">
+  <!--
   These properties must be observed by any machine
   that wants to be defined as a turtlebot. Refer
@@ -16,10 +17,9 @@
    (currently in development and awaiting feedback)
 -->
-<robot name="xacro_properties" xmlns:xacro="http://ros.org/wiki/xacro">
-<xacro:property name="cam_px" value="-0.087"/>
-<xacro:property name="cam_py" value="-0.0125" />
-<xacro:property name="cam_pz" value="0.2870" />
-<xacro:property name="cam_or" value="0" />
-<xacro:property name="cam_op" value="0" />
-<xacro:property name="cam_oy" value="0" />
+  <xacro:property name="cam_px" value="-0.087" />
+  <xacro:property name="cam_py" value="-0.0125" />
+  <xacro:property name="cam_pz" value="0.2870" />
+  <xacro:property name="cam_or" value="0" />
+  <xacro:property name="cam_op" value="0" />
+  <xacro:property name="cam_oy" value="0" />
 </robot>

File: chefbot/chefbot_description/urdf/chefbot_rviz_base.urdf.xacro (robot description, xacro)
@@ -1,3 +1,3 @@
-<?xml version="1.0" ?>
+<?xml version="1.0"?>
 <!--
   This is not a standalone urdf for kobuki. It simply defines the 'kobuki' tag that can
@@ -7,9 +7,9 @@
  -->
 <robot name="chefbot" xmlns:xacro="http://ros.org/wiki/xacro">
-  <xacro:include filename="$(find chefbot_description)/urdf/common_properties.urdf.xacro"/>
-  <xacro:include filename="$(find chefbot_description)/urdf/chefbot_base_gazebo.urdf.xacro"/>
+  <xacro:include filename="$(find chefbot_description)/urdf/common_properties.urdf.xacro" />
+  <xacro:include filename="$(find chefbot_description)/urdf/chefbot_base_gazebo.urdf.xacro" />
   <!-- Chefbot -->
   <xacro:macro name="kobuki">
-    <link name="base_footprint"/>
+    <link name="base_footprint" />
     <!--
        Base link is set at the bottom of the base mould.
@@ -23,26 +23,27 @@
     <joint name="base_joint" type="fixed">
       <origin xyz="0 0 0.0102" rpy="0 0 0" />
-      <parent link="base_footprint"/>
+      <parent link="base_footprint" />
       <child link="base_link" />
     </joint>
     <link name="base_link">
       <visual>
+        <material name="blue" />
         <geometry>
           <!-- new mesh -->
           <mesh filename="package://chefbot_description/meshes/base_plate.dae" />
         </geometry>
-<!--        <origin xyz="0.001 0 0.05199" rpy="0 0 ${M_PI/2}"/> -->
-	 <origin xyz="0.001 0 -0.034" rpy="0 0 ${M_PI/2}"/>
-      </visual>
-      <collision>
-        <geometry>
-          <cylinder length="0.10938" radius="0.178"/>
-        </geometry>
-        <origin xyz="0.0 0 0.05949" rpy="0 0 0"/>
+        <!--        <origin xyz="0.001 0 0.05199" rpy="0 0 ${M_PI/2}"/> -->
+        <origin xyz="0.001 0 -0.034" rpy="0 0 ${M_PI/2}" />
+      </visual>
+      <collision>
+        <geometry>
+          <cylinder length="0.10938" radius="0.178" />
+        </geometry>
+        <origin xyz="0.0 0 0.05949" rpy="0 0 0" />
       </collision>
       <inertial>
         <!-- COM experimentally determined -->
-        <origin xyz="0.01 0 0"/>
-        <mass value="2.4"/> <!-- 2.4/2.6 kg for small/big battery pack -->
+        <origin xyz="0.01 0 0" />
+        <mass value="2.4" /> <!-- 2.4/2.6 kg for small/big battery pack -->
         <!-- Kobuki's inertia tensor is approximated by a cylinder with homogeneous mass distribution
              More details: http://en.wikipedia.org/wiki/List_of_moment_of_inertia_tensors
@@ -52,277 +53,180 @@
              izz = 1/2 * m * r^2
           -->
-        <inertia ixx="0.019995" ixy="0.0" ixz="0.0"
-                 iyy="0.019995" iyz="0.0"
-                 izz="0.03675" />
-      </inertial>
-    </link>
-<!--
-    <joint name="wheel_left_joint" type="continuous">
-      <parent link="base_link"/>
-      <child link="chefbot_wheel_left_link"/>
-      <origin xyz="0 ${0.28/2} 0.026" rpy="${-M_PI/2} 0 0"/>
-      <axis xyz="0 0 1"/>
-    </joint>
-    <link name="chefbot_wheel_left_link">
-      <visual>
-        <geometry>
-          <mesh filename="package://chefbot_description/meshes/wheel.dae"/>
-        </geometry>
-        <origin xyz="0 0 0" rpy="0 0 0"/>
-      </visual>
-      <collision>
-        <geometry>
-          <cylinder length="0.0206" radius="0.0352"/>
-        </geometry>
-        <origin rpy="0 0 0" xyz="0 0 0"/>
-      </collision>
-      <inertial>
-        <mass value="0.01" />
-        <origin xyz="0 0 0" />
-        <inertia ixx="0.001" ixy="0.0" ixz="0.0"
-                 iyy="0.001" iyz="0.0"
-                 izz="0.001" />
-      </inertial>
-    </link>
-    <joint name="wheel_right_joint" type="continuous">
-      <parent link="base_link"/>
-      <child link="chefbot_wheel_right_link"/>
-      <origin xyz="0.00 -${0.28/2} 0.026" rpy="${-M_PI/2} 0 0"/>
-      <axis xyz="0 0 1"/>
-    </joint>
-    <link name="chefbot_wheel_right_link">
-      <visual>
-        <geometry>
-          <mesh filename="package://chefbot_description/meshes/wheel.dae"/>
-        </geometry>
-        <origin xyz="0 0 0" rpy="0 0 0"/>
-      </visual>
-      <collision>
-        <geometry>
-          <cylinder length="0.0206" radius="0.0350"/>
-        </geometry>
-        <origin rpy="0 0 0" xyz="0 0 0"/>
-      </collision>
-      <inertial>
-        <mass value="0.01" />
-        <origin xyz="0 0 0" />
-        <inertia ixx="0.001" ixy="0.0" ixz="0.0"
-                 iyy="0.001" iyz="0.0"
-                 izz="0.001" />
-      </inertial>
-    </link>
--->
-	  <link name="left_axle_link">
-	    <inertial>
-	      <origin xyz="0 -0.035 0.021"/>
-	      <mass value="0.01" />
-	      <inertia ixx="0.001" ixy="0.0" ixz="0.0"
-	        iyy="0.001" iyz="0.0" izz="0.001" />
-	    </inertial>
-	    <visual>
-	      <origin xyz="0 -0.035 0.021" rpy="0 1.5707 1.5707" />
-	      <geometry>
-            <cylinder radius="0.0045" length = "0.02"/>
-	      </geometry>
-          <material name ="light_grey" />
-	    </visual>
-	    <collision>
-	      <origin xyz="0 -0.035 0.021" rpy="0 1.5707 1.5707" />
-	      <geometry>
-            <cylinder radius="0.00635" length = "0.00635"/>
-	      </geometry>
-	    </collision>
-	  </link>
-	  <joint name="left_axle_joint" type="fixed">
-	    <origin xyz="0 0.171475 0.0178" rpy="0 0 0"/>
-	    <parent link="base_link"/>
-	    <child link="left_axle_link"/>
-	    <axis xyz="0 1 0"/>
-	  </joint>
-	  <link name="right_axle_link">
-	    <inertial>
-	      <origin xyz="0 0.035 0.021"/>
-	      <mass value="0.01" />
-	      <inertia ixx="0.001" ixy="0.0" ixz="0.0"
-	        iyy="0.001" iyz="0.0" izz="0.001" />
-	    </inertial>
-	    <visual>
-	      <origin xyz="0 0.035 0.02" rpy="0 1.5707 1.5707" />
-	      <geometry>
-            <cylinder radius="0.0045" length = "0.002"/>
-	      </geometry>
-          <material name ="light_grey" />
-	    </visual>
-	    <collision>
-	      <origin xyz="0 0.035 0.02" rpy="0 1.5707 1.5707" />
-	      <geometry>
-            <cylinder radius="0.0045" length = "0.002"/>
-	      </geometry>
-	    </collision>
-	  </link>
-	  <joint name="right_axle_joint" type="fixed">
-	    <origin xyz="0 -0.171475 0.0178" rpy="0 0 0"/>
-	    <parent link="base_link"/>
-	    <child link="right_axle_link"/>
-	    <axis xyz="0 1 0"/>
-	  </joint>
-	  <link name="left_wheel_link">
-	    <inertial>
-	      <origin xyz="0 -0.035 0.021"/>
-	      <mass value="0.01" />
-	      <inertia ixx="0.001" ixy="0.0" ixz="0.0"
-	        iyy="0.001" iyz="0.0" izz="0.001" />
-	    </inertial>
-	    <visual>
-	      <origin xyz="0 -0.035 0.021" rpy="0 1.5707 1.5707" />
-	      <geometry>
-            <cylinder radius="0.045" length = "0.02"/>
-	      </geometry>
-          <material name ="black" />
-	    </visual>
-	    <collision>
-	      <origin xyz="0 -0.035 0.021" rpy="0 1.5707 1.5707" />
-	      <geometry>
-            <cylinder radius="0.0762" length = "0.03175"/>
-	      </geometry>
-	    </collision>
-	  </link>
-        <!-- Fixed because we never rotate it anyway, it is just for show -->
-        <!-- NOTE This may prevent gazebo from working with this model -->
-	  <joint name="left_wheel_joint" type="continuous">
-	    <origin xyz="0 0.01905 0" rpy="0 0 0"/>
-	    <parent link="left_axle_link"/>
-	    <child link="left_wheel_link"/>
-	    <axis xyz="0 1 0"/>
-	  </joint>
-	  <link name="right_wheel_link">
-	    <inertial>
-	      <origin xyz="0 0.035 0.021"/>
-	      <mass value="0.01" />
-	      <inertia ixx="0.001" ixy="0.0" ixz="0.0"
-	        iyy="0.001" iyz="0.0" izz="0.001" />
-	    </inertial>
-	    <visual>
-	      <origin xyz="0 0.035 0.021" rpy="0 1.5707 1.5707" />
-	      <geometry>
-            <cylinder radius="0.045" length = "0.02"/>
-	      </geometry>
-          <material name ="black" />
-	    </visual>
-	    <collision>
-	      <origin xyz="0 0.035 0.021" rpy="0 1.5707 1.5707" />
-	      <geometry>
-            <cylinder radius="0.045" length = "0.02"/>
-	      </geometry>
-	    </collision>
-	  </link>
-        <!-- Fixed because we never rotate it anyway, it is just for show -->
-        <!-- NOTE This may prevent gazebo from working with this model -->
-	  <joint name="right_wheel_joint" type="continuous">
-	    <origin xyz="0 -0.01905 0" rpy="0 0 0"/>
-	    <parent link="right_axle_link"/>
-	    <child link="right_wheel_link"/>
-	    <axis xyz="0 1 0"/>
-	  </joint>
+        <inertia ixx="0.019995" ixy="0.0" ixz="0.0" iyy="0.019995" iyz="0.0" izz="0.03675" />
+      </inertial>
+    </link>
+    <link name="left_axle_link">
+      <inertial>
+        <origin xyz="0 -0.035 0.021" />
+        <mass value="0.01" />
+        <inertia ixx="0.001" ixy="0.0" ixz="0.0" iyy="0.001" iyz="0.0" izz="0.001" />
+      </inertial>
+      <visual>
+        <origin xyz="0 -0.035 0.021" rpy="0 1.5707 1.5707" />
+        <geometry>
+          <cylinder radius="0.0045" length="0.02" />
+        </geometry>
+        <material name="glod" />
+      </visual>
+      <collision>
+        <origin xyz="0 -0.035 0.021" rpy="0 1.5707 1.5707" />
+        <geometry>
+          <cylinder radius="0.00635" length="0.00635" />
+        </geometry>
+      </collision>
+    </link>
+    <joint name="left_axle_joint" type="fixed">
+      <origin xyz="0 0.171475 0.0178" rpy="0 0 0" />
+      <parent link="base_link" />
+      <child link="left_axle_link" />
+      <axis xyz="0 1 0" />
+    </joint>
+    <link name="right_axle_link">
+      <inertial>
+        <origin xyz="0 0.035 0.021" />
+        <mass value="0.01" />
+        <inertia ixx="0.001" ixy="0.0" ixz="0.0" iyy="0.001" iyz="0.0" izz="0.001" />
+      </inertial>
+      <visual>
+        <origin xyz="0 0.035 0.02" rpy="0 1.5707 1.5707" />
+        <geometry>
+          <cylinder radius="0.0045" length="0.002" />
+        </geometry>
+        <material name="gold" />
+      </visual>
+      <collision>
+        <origin xyz="0 0.035 0.02" rpy="0 1.5707 1.5707" />
+        <geometry>
+          <cylinder radius="0.0045" length="0.002" />
+        </geometry>
+      </collision>
+    </link>
+    <joint name="right_axle_joint" type="fixed">
+      <origin xyz="0 -0.171475 0.0178" rpy="0 0 0" />
+      <parent link="base_link" />
+      <child link="right_axle_link" />
+      <axis xyz="0 1 0" />
+    </joint>
+    <link name="left_wheel_link">
+      <inertial>
+        <origin xyz="0 -0.035 0.021" />
+        <mass value="0.01" />
+        <inertia ixx="0.001" ixy="0.0" ixz="0.0" iyy="0.001" iyz="0.0" izz="0.001" />
+      </inertial>
+      <visual>
+        <origin xyz="0 -0.035 0.021" rpy="0 1.5707 1.5707" />
+        <geometry>
+          <cylinder radius="0.045" length="0.02" />
+        </geometry>
+        <material name="black" />
+      </visual>
+      <collision>
+        <origin xyz="0 -0.035 0.021" rpy="0 1.5707 1.5707" />
+        <geometry>
+          <cylinder radius="0.0762" length="0.03175" />
+        </geometry>
+      </collision>
+    </link>
+    <!-- Fixed because we never rotate it anyway, it is just for show -->
+    <!-- NOTE This may prevent gazebo from working with this model -->
+    <joint name="left_wheel_joint" type="continuous">
+      <origin xyz="0 0.01905 0" rpy="0 0 0" />
+      <parent link="left_axle_link" />
+      <child link="left_wheel_link" />
+      <axis xyz="0 1 0" />
+    </joint>
+    <link name="right_wheel_link">
+      <inertial>
+        <origin xyz="0 0.035 0.021" />
+        <mass value="0.01" />
+        <inertia ixx="0.001" ixy="0.0" ixz="0.0" iyy="0.001" iyz="0.0" izz="0.001" />
+      </inertial>
+      <visual>
+        <origin xyz="0 0.035 0.021" rpy="0 1.5707 1.5707" />
+        <geometry>
+          <cylinder radius="0.045" length="0.02" />
+        </geometry>
+        <material name="black" />
+      </visual>
+      <collision>
+        <origin xyz="0 0.035 0.021" rpy="0 1.5707 1.5707" />
+        <geometry>
+          <cylinder radius="0.045" length="0.02" />
+        </geometry>
+      </collision>
+    </link>
+    <!-- Fixed because we never rotate it anyway, it is just for show -->
+    <!-- NOTE This may prevent gazebo from working with this model -->
+    <joint name="right_wheel_joint" type="continuous">
+      <origin xyz="0 -0.01905 0" rpy="0 0 0" />
+      <parent link="right_axle_link" />
+      <child link="right_wheel_link" />
+      <axis xyz="0 1 0" />
+    </joint>
     <joint name="caster_front_joint" type="fixed">
-      <parent link="base_link"/>
-      <child link="chefbot_caster_front_link"/>
-      <origin xyz="0.115 0.0 0.007" rpy="${-M_PI/2} 0 0"/>
+      <parent link="base_link" />
+      <child link="chefbot_caster_front_link" />
+      <origin xyz="0.115 0.0 0.007" rpy="${-M_PI/2} 0 0" />
     </joint>
     <link name="chefbot_caster_front_link">
       <collision>
         <geometry>
-          <cylinder length="0.0176" radius="0.017"/>
-        </geometry>
-        <origin rpy="0 0 0" xyz="0 0 0"/>
-      </collision>
-      <inertial>
-        <mass value="0.01" />
-        <origin xyz="0 0 0" />
-        <inertia ixx="0.001" ixy="0.0" ixz="0.0"
-                 iyy="0.001" iyz="0.0"
-                 izz="0.001" />
-      </inertial>
+          <cylinder length="0.0176" radius="0.017" />
+        </geometry>
+        <origin rpy="0 0 0" xyz="0 0 0" />
+      </collision>
+      <xacro:default_inertial z_value="0" i_value="0.001" mass="0.01" />
     </link>
     <joint name="chefbot_caster_back_joint" type="fixed">
-      <parent link="base_link"/>
-      <child link="chefbot_caster_back_link"/>
-      <origin xyz="-0.135 0.0 0.009" rpy="${-M_PI/2} 0 0"/>
+      <parent link="base_link" />
+      <child link="chefbot_caster_back_link" />
+      <origin xyz="-0.135 0.0 0.009" rpy="${-M_PI/2} 0 0" />
     </joint>
     <link name="chefbot_caster_back_link">
       <collision>
         <geometry>
-          <cylinder length="0.0176" radius="0.017"/>
-        </geometry>
-        <origin rpy="0 0 0" xyz="0 0 0"/>
-      </collision>
-      <inertial>
-        <mass value="0.01" />
-        <origin xyz="0 0 0" />
-        <inertia ixx="0.001" ixy="0.0" ixz="0.0"
-                 iyy="0.001" iyz="0.0"
-                 izz="0.001" />
-      </inertial>
+          <cylinder length="0.0176" radius="0.017" />
+        </geometry>
+        <origin rpy="0 0 0" xyz="0 0 0" />
+      </collision>
+      <xacro:default_inertial z_value="0" i_value="0.001" mass="0.01" />
     </link>
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
File: chefbot/chefbot_description/urdf/chefbot_rviz_library.urdf.xacro (robot description, xacro)
@@ -1,22 +1,30 @@
 <?xml version="1.0"?>
 <robot name="chefbot" xmlns:xacro="http://ros.org/wiki/xacro">
-<!--
+  <!--
   The complete turtlebot library of xacros for easy reference
  -->
   <!-- General -->
-  <xacro:include filename="$(find chefbot_description)/urdf/common_properties.urdf.xacro"/>
-  <xacro:include filename="$(find chefbot_description)/urdf/chefbot_properties.urdf.xacro"/>
-<!-- Need changes in chefbot base and circle -->
+  <xacro:include filename="$(find chefbot_description)/urdf/common_properties.urdf.xacro" />
+  <xacro:include filename="$(find chefbot_description)/urdf/chefbot_properties.urdf.xacro" />
+  <xacro:include filename="$(find chefbot_description)/urdf/materials.xacro" />
+  <xacro:macro name="default_inertial" params="z_value i_value mass">
+    <inertial>
+      <origin xyz="0 0 ${z_value}" rpy="0 0 0" />
+      <mass value="${mass}" />
+      <inertia ixx="${i_value}" ixy="0.0" ixz="0.0" iyy="${i_value}" iyz="0.0" izz="${i_value}" />
+    </inertial>
+  </xacro:macro>
+  <!-- Need changes in chefbot base and circle -->
   <!-- Bases -->
-  <xacro:include filename="$(find chefbot_description)/urdf/chefbot_rviz_base.urdf.xacro"/>
-<!--  <xacro:include filename="$(find create_description)/urdf/create.urdf.xacro"/>
+  <xacro:include filename="$(find chefbot_description)/urdf/chefbot_rviz_base.urdf.xacro" />
+  <!--  <xacro:include filename="$(find create_description)/urdf/create.urdf.xacro"/>
   <xacro:include filename="$(find kobuki_description)/urdf/kobuki.urdf.xacro" />
 -->
   <!-- Stacks -->
-<!--  <xacro:include filename="$(find chefbot_description)/urdf/circles.urdf.xacro"/>  -->
-<!-- <xacro:include filename="$(find chefbot_description)/urdf/stacks/circles.urdf.xacro"/> -->
-<!--  <xacro:include filename="$(find turtlebot_description)/urdf/stacks/hexagons.urdf.xacro"/> -->
+  <!--  <xacro:include filename="$(find chefbot_description)/urdf/circles.urdf.xacro"/>  -->
+  <!-- <xacro:include filename="$(find chefbot_description)/urdf/stacks/circles.urdf.xacro"/> -->
+  <!--  <xacro:include filename="$(find turtlebot_description)/urdf/stacks/hexagons.urdf.xacro"/> -->
   <!-- 3D Sensors -->
-  <xacro:include filename="$(find chefbot_description)/urdf/sensors/kinect.urdf.xacro"/>
-  <xacro:include filename="$(find chefbot_description)/urdf/sensors/asus_xtion_pro.urdf.xacro"/>
+  <xacro:include filename="$(find chefbot_description)/urdf/sensors/kinect.urdf.xacro" />
+  <xacro:include filename="$(find chefbot_description)/urdf/sensors/asus_xtion_pro.urdf.xacro" />
 </robot>
