Commit message: amend xacro

File: chefbot/chefbot_description/urdf/chefbot_properties.urdf.xacro (robot description, xacro)
@@ -23,3 +23,20 @@
   <xacro:property name="cam_op" value="0" />
   <xacro:property name="cam_oy" value="0" />
+  <!-- PROPERTY LIST -->
+  <!--All units in m-kg-s-radians unit system -->
+  <xacro:property name="M_PI" value="3.1415926535897931" />
+  <xacro:property name="M_PI_2" value="1.570796327" />
+  <xacro:property name="DEG_TO_RAD" value="0.017453293" />
+  <!-- Main body radius and height -->
+  <!-- Main Body Cylinder base   -->
+  <xacro:property name="base_height" value="0.02" />
+  <xacro:property name="base_radius" value="0.15" />
+  <xacro:property name="base_mass" value="4.0" /> <!-- in kg-->
+  <!-- Wheels -->
+  <xacro:property name="wheel_radius" value="0.04" />
+  <xacro:property name="wheel_height" value="0.02" />
+  <xacro:property name="wheel_mass" value="2.5" /> <!-- in kg-->
+  <xacro:property name="base_x_origin_to_wheel_origin" value="0.25" />
+  <xacro:property name="base_y_origin_to_wheel_origin" value="0.3" />
+  <xacro:property name="base_z_origin_to_wheel_origin" value="0.0" />
 </robot>

File: chefbot/chefbot_description/urdf/chefbot_rviz_base.urdf.xacro (robot description, xacro)
@@ -110,5 +110,5 @@
     <link name="left_wheel_link">
       <inertial>
-        <origin xyz="0 -0.035 0.021" />
+        <origin xyz="0 -0.035 0.021" rpy="0 1.5707 1.5707"/>
         <mass value="0.01" />
         <inertia ixx="0.001" ixy="0.0" ixz="0.0" iyy="0.001" iyz="0.0" izz="0.001" />

File: chefbot/chefbot_description/urdf/chefbot_rviz_library.urdf.xacro (robot description, xacro)
@@ -8,11 +8,4 @@
   <xacro:include filename="$(find chefbot_description)/urdf/chefbot_properties.urdf.xacro" />
   <xacro:include filename="$(find chefbot_description)/urdf/materials.xacro" />
-  <xacro:macro name="default_inertial" params="z_value i_value mass">
-    <inertial>
-      <origin xyz="0 0 ${z_value}" rpy="0 0 0" />
-      <mass value="${mass}" />
-      <inertia ixx="${i_value}" ixy="0.0" ixz="0.0" iyy="${i_value}" iyz="0.0" izz="${i_value}" />
-    </inertial>
-  </xacro:macro>
   <!-- Need changes in chefbot base and circle -->
   <!-- Bases -->

Commit message: robot_state_pub add param robot_description

File: chefbot/chefbot_description/urdf/chefbot_properties.urdf.xacro (robot description, xacro)
@@ -1,4 +1,4 @@
 <?xml version="1.0"?>
-<robot xmlns:xacro="http://ros.org/wiki/xacro">
+<robot xmlns:xacro="http://ros.org/wiki/xacro" name="roachbot">
   <!--
   These properties must be observed by any machine
@@ -25,18 +25,25 @@
   <!-- PROPERTY LIST -->
   <!--All units in m-kg-s-radians unit system -->
-  <xacro:property name="M_PI" value="3.1415926535897931" />
-  <xacro:property name="M_PI_2" value="1.570796327" />
+  <xacro:property name="M_PI_2" value="${pi/2}" />
   <xacro:property name="DEG_TO_RAD" value="0.017453293" />
   <!-- Main body radius and height -->
   <!-- Main Body Cylinder base   -->
+  <xacro:property name="base_width" value="0.16"/>
+  <xacro:property name="base_len" value="0.16"/>
   <xacro:property name="base_height" value="0.02" />
-  <xacro:property name="base_radius" value="0.15" />
+  <xacro:property name="base_radius" value="0.07" />
   <xacro:property name="base_mass" value="4.0" /> <!-- in kg-->
+  <xacro:property name="wheel_separation" value="${2*(wheel_radius+0.5*wheel_thick)"/>
+  <xacro:property name="wheel_thick" value="0.01"/>
+  <xacro:property name="base_wheel_gap" value="0.007"/>
   <!-- Wheels -->
-  <xacro:property name="wheel_radius" value="0.04" />
-  <xacro:property name="wheel_height" value="0.02" />
-  <xacro:property name="wheel_mass" value="2.5" /> <!-- in kg-->
+  <xacro:property name="wheel_radius" value="0.035" />
+  <xacro:property name="wheel_mass" value="0.5" /> <!-- in kg-->
+  <xacro:property name="wheel_joint_offset" value="0.02"/>
   <xacro:property name="base_x_origin_to_wheel_origin" value="0.25" />
   <xacro:property name="base_y_origin_to_wheel_origin" value="0.3" />
   <xacro:property name="base_z_origin_to_wheel_origin" value="0.0" />
+  <xacro:property name="caster_wheel_radius" value="${(wheel_radius - base_height/2)/2}"/>
+  <xacro:property name="caster_wheel_mass" value="0.01"/>
+  <xacro:property name="caster_wheel_joint_offset" value="-0.052"/>
 </robot>

File: chefbot/chefbot_description/urdf/diff_wheeled_robot.xacro (robot description, xacro)
@@ -1,17 +1,17 @@
 <?xml version="1.0"?>
 <robot name="differential_wheeled_robot" xmlns:xacro="http://ros.org/wiki/xacro">
-  <xacro:include filename="$(find mastering_ros_robot_description_pkg)/urdf/wheel.urdf.xacro" />
-<!-- Defining the colors used in this robot -->
+  <xacro:include filename="$(find chefbot_description)/urdf/wheel.urdf.xacro" />
+  <!-- Defining the colors used in this robot -->
   <material name="Black">
-    <color rgba="0.0 0.0 0.0 1.0"/>
+    <color rgba="0.0 0.0 0.0 1.0" />
   </material>
   <material name="Red">
-    <color rgba="0.8 0.0 0.0 1.0"/>
+    <color rgba="0.8 0.0 0.0 1.0" />
   </material>
   <material name="White">
-    <color rgba="1.0 1.0 1.0 1.0"/>
+    <color rgba="1.0 1.0 1.0 1.0" />
   </material>
   <material name="Blue">
-    <color rgba="0.0 0.0 0.8 1.0"/>
+    <color rgba="0.0 0.0 0.8 1.0" />
   </material>
   <!-- PROPERTY LIST -->
@@ -36,5 +36,6 @@
   <xacro:property name="caster_b_mass" value="0.5" /> <!-- in kg-->
   <!-- Wheels -->
-  <xacro:property name="wheel_mass" value="2.5" /> --> <!-- in kg-->
+  <xacro:property name="wheel_mass" value="2.5" />
+  --> <!-- in kg-->
   <xacro:property name="base_x_origin_to_wheel_origin" value="0.25" />
   <xacro:property name="base_y_origin_to_wheel_origin" value="0.3" />
@@ -44,7 +45,5 @@
   <!-- Macro for calculating inertia of cylinder -->
   <xacro:macro name="cylinder_inertia" params="m r h">
-    <inertia  ixx="${m*(3*r*r+h*h)/12}" ixy = "0" ixz = "0"
-              iyy="${m*(3*r*r+h*h)/12}" iyz = "0"
-              izz="${m*r*r/2}" />
+    <inertia ixx="${m*(3*r*r+h*h)/12}" ixy="0" ixz="0" iyy="${m*(3*r*r+h*h)/12}" iyz="0" izz="${m*r*r/2}" />
   </xacro:macro>
   <!-- BASE-FOOTPRINT -->
@@ -54,13 +53,11 @@
       <mass value="0.0001" />
       <origin xyz="0 0 0" />
-      <inertia ixx="0.0001" ixy="0.0" ixz="0.0"
-          iyy="0.0001" iyz="0.0"
-          izz="0.0001" />
+      <inertia ixx="0.0001" ixy="0.0" ixz="0.0" iyy="0.0001" iyz="0.0" izz="0.0001" />
     </inertial>
     <visual>
-        <origin xyz="0 0 0" rpy="0 0 0" />
-        <geometry>
-            <box size="0.001 0.001 0.001" />
-        </geometry>
+      <origin xyz="0 0 0" rpy="0 0 0" />
+      <geometry>
+        <box size="0.001 0.001 0.001" />
+      </geometry>
     </visual>
   </link>
@@ -70,5 +67,5 @@
   <joint name="base_footprint_joint" type="fixed">
     <origin xyz="0 0 ${wheel_radius - base_z_origin_to_wheel_origin}" rpy="0 0 0" />
-    <parent link="base_footprint"/>
+    <parent link="base_footprint" />
     <child link="base_link" />
   </joint>
@@ -77,13 +74,11 @@
       <mass value="${base_mass}" />
       <origin xyz="0 0 0" />
-      <inertia ixx="0.0001" ixy="0.0" ixz="0.0"
-          iyy="0.0001" iyz="0.0"
-          izz="0.0001" />
-      <cylinder_inertia  m="${base_mass}" r="${base_radius}" h="${base_height}" />
+      <inertia ixx="0.0001" ixy="0.0" ixz="0.0" iyy="0.0001" iyz="0.0" izz="0.0001" />
+      <cylinder_inertia m="${base_mass}" r="${base_radius}" h="${base_height}" />
     </inertial>
     <visual>
       <origin xyz="0 0 0" rpy="0 0 0" />
       <geometry>
-          <cylinder length="${base_height}" radius="${base_radius}" />
+        <cylinder length="${base_height}" radius="${base_radius}" />
       </geometry>
       <material name="White" />
@@ -92,5 +87,5 @@
       <origin xyz="0 0 0" rpy="0 0 0 " />
       <geometry>
-          <cylinder length="${base_height}" radius="${base_radius}" />
+        <cylinder length="${base_height}" radius="${base_radius}" />
       </geometry>
     </collision>
@@ -104,5 +99,5 @@
       <origin xyz="0 0.02 0" rpy="${M_PI/2} 0 0" />
       <geometry>
-				<sphere radius="${caster_f_radius}" />
+        <sphere radius="${caster_f_radius}" />
       </geometry>
       <material name="Black" />
@@ -110,20 +105,18 @@
     <collision>
       <geometry>
-				<sphere radius="${caster_f_radius}" />
+        <sphere radius="${caster_f_radius}" />
       </geometry>
-    <origin xyz="0 0.02 0" rpy="${M_PI/2} 0 0" />
+      <origin xyz="0 0.02 0" rpy="${M_PI/2} 0 0" />
     </collision>
     <inertial>
       <mass value="${caster_f_mass}" />
       <origin xyz="0 0 0" />
-      <inertia ixx="0.001" ixy="0.0" ixz="0.0"
-               iyy="0.001" iyz="0.0"
-               izz="0.001" />
+      <inertia ixx="0.001" ixy="0.0" ixz="0.0" iyy="0.001" iyz="0.0" izz="0.001" />
     </inertial>
   </link>
-	<joint name="caster_front_joint" type="fixed">
-    <parent link="base_link"/>
-    <child link="caster_front_link"/>
-    <origin xyz="0.115 0.0 0.007" rpy="${-M_PI/2} 0 0"/>
+  <joint name="caster_front_joint" type="fixed">
+    <parent link="base_link" />
+    <child link="caster_front_link" />
+    <origin xyz="0.115 0.0 0.007" rpy="${-M_PI/2} 0 0" />
   </joint>
   <gazebo reference="caster_front_link">
@@ -131,57 +124,55 @@
   </gazebo>
   <link name="caster_back_link">
-  <visual>
-    <origin xyz="0.02 0.02 0 " rpy="${M_PI/2} 0 0" />
-    <geometry>
-			<sphere radius="${caster_b_radius}" />
-    </geometry>
-    <material name="Black" />
-  </visual>
-  <collision>
-    <geometry>
-			<sphere radius="${caster_b_radius}" />
-     </geometry>
-     <origin xyz="0 0.02 0 " rpy="${M_PI/2} 0 0" />
+    <visual>
+      <origin xyz="0.02 0.02 0 " rpy="${M_PI/2} 0 0" />
+      <geometry>
+        <sphere radius="${caster_b_radius}" />
+      </geometry>
+      <material name="Black" />
+    </visual>
+    <collision>
+      <geometry>
+        <sphere radius="${caster_b_radius}" />
+      </geometry>
+      <origin xyz="0 0.02 0 " rpy="${M_PI/2} 0 0" />
     </collision>
     <inertial>
       <mass value="${caster_b_mass}" />
       <origin xyz="0 0 0" />
-      <inertia ixx="0.001" ixy="0.0" ixz="0.0"
-               iyy="0.001" iyz="0.0"
-               izz="0.001" />
+      <inertia ixx="0.001" ixy="0.0" ixz="0.0" iyy="0.001" iyz="0.0" izz="0.001" />
     </inertial>
   </link>
   <joint name="caster_back_joint" type="fixed">
-    <parent link="base_link"/>
-    <child link="caster_back_link"/>
-    <origin xyz="-0.135 0.0 0.009" rpy="${-M_PI/2} 0 0"/>
+    <parent link="base_link" />
+    <child link="caster_back_link" />
+    <origin xyz="-0.135 0.0 0.009" rpy="${-M_PI/2} 0 0" />
   </joint>
   <gazebo reference="caster_back_link">
-   <turnGravityOff>false</turnGravityOff>
+    <turnGravityOff>false</turnGravityOff>
   </gazebo>
-  <xacro:wheel fb="front" lr="right" parent="base_link" translateX="0" translateY="-0.5" flipY="1"/>
-	<xacro:wheel fb="front" lr="left" parent="base_link" translateX="0" translateY="0.5" flipY="1"/>
-	<gazebo>
-  	<plugin name="differential_drive_controller" filename="libgazebo_ros_diff_drive.so">
-	    <legacyMode>true</legacyMode>
-	    <rosDebugLevel>Debug</rosDebugLevel>
-	    <publishWheelTF>false</publishWheelTF>
-	    <robotNamespace>/</robotNamespace>
-	    <publishTf>1</publishTf>
-	    <publishWheelJointState>false</publishWheelJointState>
-	    <alwaysOn>true</alwaysOn>
-	    <updateRate>100.0</updateRate>
-	    <leftJoint>front_left_wheel_joint</leftJoint>
-	    <rightJoint>front_right_wheel_joint</rightJoint>
-	    <wheelSeparation>${2*base_radius}</wheelSeparation>
-	    <wheelDiameter>${2*wheel_radius}</wheelDiameter>
-	    <broadcastTF>1</broadcastTF>
-	    <wheelTorque>30</wheelTorque>
-	    <wheelAcceleration>1.8</wheelAcceleration>
-	    <commandTopic>cmd_vel</commandTopic>
-	    <odometryFrame>odom</odometryFrame>
-	    <odometryTopic>odom</odometryTopic>
-	    <robotBaseFrame>base_footprint</robotBaseFrame>
-   </plugin>
+  <xacro:wheel fb="front" lr="right" parent="base_link" translateX="0" translateY="-0.5" flipY="1" />
+  <xacro:wheel fb="front" lr="left" parent="base_link" translateX="0" translateY="0.5" flipY="1" />
+  <gazebo>
+    <plugin name="differential_drive_controller" filename="libgazebo_ros_diff_drive.so">
+      <legacyMode>true</legacyMode>
+      <rosDebugLevel>Debug</rosDebugLevel>
+      <publishWheelTF>false</publishWheelTF>
+      <robotNamespace>/</robotNamespace>
+      <publishTf>1</publishTf>
+      <publishWheelJointState>false</publishWheelJointState>
+      <alwaysOn>true</alwaysOn>
+      <updateRate>100.0</updateRate>
+      <leftJoint>front_left_wheel_joint</leftJoint>
+      <rightJoint>front_right_wheel_joint</rightJoint>
+      <wheelSeparation>${2*base_radius}</wheelSeparation>
+      <wheelDiameter>${2*wheel_radius}</wheelDiameter>
+      <broadcastTF>1</broadcastTF>
+      <wheelTorque>30</wheelTorque>
+      <wheelAcceleration>1.8</wheelAcceleration>
+      <commandTopic>cmd_vel</commandTopic>
+      <odometryFrame>odom</odometryFrame>
+      <odometryTopic>odom</odometryTopic>
+      <robotBaseFrame>base_footprint</robotBaseFrame>
+    </plugin>
   </gazebo>
 </robot>

File: chefbot/chefbot_description/urdf/materials.xacro (robot description, xacro)
@@ -1,10 +1,4 @@
 <?xml version="1.0"?>
-<robot>
-    <material name="black">
-        <color rgba="0.0 0.0 0.0 1.0" />
-    </material>
-    <material name="blue">
-        <color rgba="0.0 0.0 0.8 1.0" />
-    </material>
+<robot xmlns:xacro="http://www.ros.org/wiki/xacro" name="roachbot">
     <material name="green">
         <color rgba="0.0 1.0 0.0 1.0" />
@@ -22,6 +16,12 @@
         <color rgba="0.8 0.0 0.0 1.0" />
     </material>
+    <material name="black">
+        <color rgba="0 0 0 1" />
+    </material>
     <material name="white">
-        <color rgba="1.0 1.0 1.0 1.0" />
+        <color rgba="1 1 1 1" />
+    </material>
+    <material name="blue">
+        <color rgba="0 0 0.8 1" />
     </material>
     <material name="gold">

File: chefbot/chefbot_description/urdf/rbot.xacro (robot description, xacro)
@@ -10,5 +10,5 @@
     <!-- <xacro:include filename="$(find chefbot_description)/urdf/rbot.gazebo" /> -->
     <xacro:include filename="$(find chefbot_description)/urdf/macros.xacro" />
-    <link name="base_footprint" />
+    <link name="base_footprint"/>
     <!--
        Base link is set at the bottom of the base mould.
@@ -21,5 +21,4 @@
       -->
     <joint name="base_joint" type="fixed">
-        <origin xyz="0 0 0.0102" rpy="0 0 0" />
         <parent link="base_footprint" />
         <child link="base_link" />
@@ -27,11 +26,10 @@
     <link name="base_link">
         <visual>
-            <material name="blue" />
             <geometry>
                 <!-- new mesh -->
                 <mesh filename="package://chefbot_description/meshes/base_plate.dae" />
             </geometry>
-            <!--        <origin xyz="0.001 0 0.05199" rpy="0 0 ${M_PI/2}"/> -->
-            <origin xyz="0.001 0 -0.034" rpy="0 0 ${M_PI/2}" />
+            <!--        <origin xyz="0.001 0 0.05199" rpy="0 0 ${M_PI_2}"/> -->
+            <origin xyz="0.001 0 -0.034" rpy="0 0 ${M_PI_2}" />
         </visual>
         <collision>
@@ -55,4 +53,5 @@
         </inertial>
     </link>
+    <!--
     <link name="left_axle_link">
         <inertial>
@@ -107,8 +106,9 @@
         <axis xyz="0 1 0" />
     </joint>
+-->
     <joint name="caster_front_joint" type="fixed">
         <parent link="base_link" />
         <child link="chefbot_caster_front_link" />
-        <origin xyz="0.115 0.0 0.007" rpy="${-M_PI/2} 0 0" />
+        <origin xyz="0.115 0.0 0.007" rpy="${-M_PI_2} 0 0" />
     </joint>
     <link name="chefbot_caster_front_link">
@@ -124,5 +124,5 @@
         <parent link="base_link" />
         <child link="chefbot_caster_back_link" />
-        <origin xyz="-0.135 0.0 0.009" rpy="${-M_PI/2} 0 0" />
+        <origin xyz="-0.135 0.0 0.009" rpy="${-M_PI_2} 0 0" />
     </joint>
     <link name="chefbot_caster_back_link">
@@ -146,5 +146,5 @@
     </link>
     <joint name="cliff_sensor_left_joint" type="fixed">
-        <origin xyz="0.08734 0.13601 0.0214" rpy="0 ${M_PI/2} 0" />
+        <origin xyz="0.08734 0.13601 0.0214" rpy="0 ${M_PI_2} 0" />
         <parent link="base_link" />
         <child link="cliff_sensor_left_link" />
@@ -154,5 +154,5 @@
     </link>
     <joint name="cliff_sensor_right_joint" type="fixed">
-        <origin xyz="0.085 -0.13601 0.0214" rpy="0 ${M_PI/2} 0" />
+        <origin xyz="0.085 -0.13601 0.0214" rpy="0 ${M_PI_2} 0" />
         <parent link="base_link" />
         <child link="cliff_sensor_right_link" />
@@ -162,5 +162,5 @@
     </link>
     <joint name="cliff_sensor_front_joint" type="fixed">
-        <origin xyz="0.156 0.00 0.0214" rpy="0 ${M_PI/2} 0" />
+        <origin xyz="0.156 0.00 0.0214" rpy="0 ${M_PI_2} 0" />
         <parent link="base_link" />
         <child link="cliff_sensor_front_link" />
@@ -169,8 +169,12 @@
         <xacro:default_inertial z_value="0" i_value="0.001" mass="0.01" />
     </link>
+    <xacro:wheel prefix="left" reflect="1" />
+    <xacro:wheel prefix="right" reflect="-1" />
+    <!--
     <xacro:link_wheel lr="left" flipY="1" />
     <xacro:joint_wheel name="left_wheel_joint" parent="left_axle_link" child="left_wheel_link" origin_xyz="0 0 0" />
     <xacro:link_wheel lr="right" flipY="1" />
     <xacro:joint_wheel name="right_wheel_joint" parent="right_axle_link" child="right_wheel_link" origin_xyz="0 0 0" />
+-->
     <!-- transmission -->
     <transmission name="left_wheel_joint_trans">

File: chefbot/chefbot_description/urdf/wheel.urdf.xacro (robot description, xacro)
@@ -54,5 +54,5 @@
       <actuator name="${fb}_${lr}_wheel_joint_motor">
         <hardwareInterface>EffortJointInterface</hardwareInterface>
-        <mechanicalReduction>1</mechanicalReduction>
+        <mechanicalReduction>10</mechanicalReduction>
       </actuator>
     </transmission>
