Commit message: add rviz

File: chefbot/chefbot_description/urdf/properties.xacro (robot description, xacro)
@@ -43,5 +43,5 @@
   <xacro:property name='lidar_height' value='0.04'/>
   <!-- Wheels -->
-  <xacro:property name="wheel_radius" value="0.035" />
+  <xacro:property name="wheel_radius" value="0.034" />
   <xacro:property name="wheel_thick" value="0.01" />
   <xacro:property name="wheel_mass" value="0.5" /> <!-- in kg-->

Commit message: serialdataGateway init bugfix

File: chefbot/chefbot_description/urdf/properties.xacro (robot description, xacro)
@@ -54,4 +54,3 @@
   <xacro:property name="cameraSize" value="0.05" />
   <xacro:property name="cameraMass" value="0.1" />
-  <xacro:property name="DEG_TO_RAD" value="0.017453293" />
 </robot>
