Commit message: refine launch files

File: chefbot/chefbot_description/urdf/kbot.xacro (robot description, xacro)
@@ -11,5 +11,4 @@
     -->
   <link name="base_footprint">
-    <!--
         <xacro:box_inertia m="20" w="0.001" h="0.001" d="0.001" />
         <visual>
@@ -19,8 +18,6 @@
             </geometry>
         </visual>
-      -->
   </link>
   <link name="base_link">
-    <xacro:cylinder_inertia m="${base_mass}" r="${base_radius}" h="${base_height}" />
     <visual>
       <geometry>
@@ -34,8 +31,8 @@
       </geometry>
     </collision>
+    <xacro:cylinder_inertia m="${base_mass}" r="${base_radius}" h="${base_height}" />
   </link>
   <joint name="base_link_joint" type="fixed">
     <origin xyz="0 0 ${base_radius}" rpy="0 0 0" />
-    -->
     <parent link="base_footprint" />
     <child link="base_link" />
@@ -69,11 +66,12 @@
       <origin xyz="0 0 0" rpy="0 0 0" />
       <geometry>
-        <cylinder radius="${hokuyo_size}" length="0.04" />
+        <cylinder radius="${lidar_radius}" length="${lidar_height}" />
       </geometry>
       <material name="blue" />
     </visual>
+    <xacro:cylinder_inertia m="${lidar_mass}" r="${lidar_radius}" h="${lidar_height}" />
   </link>
   <joint name="hokuyo_joint" type="fixed">
-    <origin xyz="0 0 ${base_height+hokuyo_size/4}" rpy="0 0 0" />
+    <origin xyz="0 0 ${base_height+lidar_radius/4}" rpy="0 0 0" />
     <parent link="base_link" />
     <child link="laser_link" />

File: chefbot/chefbot_description/urdf/properties.xacro (robot description, xacro)
@@ -38,5 +38,8 @@
   <xacro:property name="wheel_separation" value="${2*(wheel_radius+0.5*wheel_thick)" />
   <xacro:property name="wheel_thick" value="0.01" />
-  <xacro:property name="base_wheel_gap" value="${base_radius*0.15}" />
+  <xacro:property name="base_wheel_gap" value="${base_radius*0.12}" />
+  <xacro:property name='lidar_mass' value='0.125'/>
+  <xacro:property name='lidar_radius' value='0.03'/>
+  <xacro:property name='lidar_height' value='0.04'/>
   <!-- Wheels -->
   <xacro:property name="wheel_radius" value="0.035" />

Commit message: speed_message from %d to %f (bugfix)

File: chefbot/chefbot_description/urdf/kbot.xacro (robot description, xacro)
@@ -11,11 +11,13 @@
     -->
   <link name="base_footprint">
-        <xacro:box_inertia m="20" w="0.001" h="0.001" d="0.001" />
-        <visual>
-            <origin xyz="0 0 0" rpy="0 0 0" />
-            <geometry>
-                <box size="0.001 0.001 0.001" />
-            </geometry>
-        </visual>
+    <!--
+    <xacro:box_inertia m="0.0001" w="0.001" h="0.001" d="0.001" />
+    <visual>
+      <origin xyz="0 0 0" rpy="0 0 0" />
+      <geometry>
+        <box size="0.001 0.001 0.001" />
+      </geometry>
+    </visual>
+  -->
   </link>
   <link name="base_link">

Commit message: add an additional caster

File: chefbot/chefbot_description/urdf/kbot.xacro (robot description, xacro)
@@ -40,28 +40,8 @@
     <child link="base_link" />
   </joint>
-  <link name="caster_wheel">
-    <visual>
-      <origin xyz="0 0 0" rpy="0 0 0" />
-      <geometry>
-        <sphere radius="${caster_wheel_radius}" />
-      </geometry>
-      <material name="white" />
-    </visual>
-    <collision>
-      <origin xyz="0 0 0" rpy="0 0 0" />
-      <geometry>
-        <sphere radius="${caster_wheel_radius}" />
-      </geometry>
-    </collision>
-    <xacro:sphere_inertia m="${caster_wheel_mass}" r="${caster_wheel_radius}" />
-  </link>
-  <joint name="caster_wheel_joint" type="fixed">
-    <axis xyz="0 1 0" rpy="0 0 0" />
-    <parent link="base_link" />
-    <child link="caster_wheel" />
-    <origin xyz="${caster_wheel_joint_offset} 0 -${caster_wheel_radius}" rpy="0 0 0" />
-  </joint>
   <xacro:wheel prefix="left" reflect="1" />
   <xacro:wheel prefix="right" reflect="-1" />
+  <xacro:caster prefix="front" reflect="-1" />
+  <xacro:caster prefix="rear" reflect="1" />
   <link name="laser_link">
     <visual>

File: chefbot/chefbot_description/urdf/kbot_macros.xacro (robot description, xacro)
@@ -71,4 +71,28 @@
         </xacro:if>
     </xacro:macro>
+    <xacro:macro name="caster" params="prefix reflect">
+        <link name="${prefix}_caster_wheel">
+            <visual>
+                <origin xyz="0 0 0" rpy="0 0 0" />
+                <geometry>
+                    <sphere radius="${caster_wheel_radius}" />
+                </geometry>
+                <material name="white" />
+            </visual>
+            <collision>
+                <origin xyz="0 0 0" rpy="0 0 0" />
+                <geometry>
+                    <sphere radius="${caster_wheel_radius}" />
+                </geometry>
+            </collision>
+            <xacro:sphere_inertia m="${caster_wheel_mass}" r="${caster_wheel_radius}" />
+        </link>
+        <joint name="${prefix}_caster_wheel_joint" type="fixed">
+            <axis xyz="0 1 0" rpy="0 0 0" />
+            <parent link="base_link" />
+            <child link="${prefix}_caster_wheel" />
+            <origin xyz="${reflect*caster_wheel_joint_offset} 0 -${caster_wheel_radius}" rpy="0 0 0" />
+        </joint>
+    </xacro:macro>
     <!--
     <xacro:macro name="joint_wheel" params="name child parent origin_xyz">

Commit message: add imu in xacro

File: chefbot/chefbot_description/urdf/kbot.xacro (robot description, xacro)
@@ -57,4 +57,10 @@
     <child link="laser_link" />
   </joint>
+  <link name="imu"/>
+  <joint name="imu_joint" type="fixed">
+    <origin rpy="${pi} 0 0" xyz="-0.035.03 0.2"/>
+    <parent link="base_link" />
+    <child link="imu"/>
+  </joint>
   <!--
     <link name="camera">

Commit message: fix urdf bug to make it show right direction in rviz

File: chefbot/chefbot_description/urdf/kbot.xacro (robot description, xacro)
@@ -10,13 +10,4 @@
        add a simple link without inertia and make a joint between it and the chassis
     -->
-  <link name="base_footprint">
-    <xacro:box_inertia m="0.0001" w="0.001" h="0.001" d="0.001" />
-    <visual>
-      <origin xyz="0 0 0" rpy="0 0 0" />
-      <geometry>
-        <box size="0.001 0.001 0.001" />
-      </geometry>
-    </visual>
-  </link>
   <link name="base_link">
     <visual>
@@ -33,13 +24,16 @@
     <xacro:cylinder_inertia m="${base_mass}" r="${base_radius}" h="${base_height}" />
   </link>
+  <link name="base_footprint">
+    <xacro:box_inertia m="0" w="0" h="0" d="0" />
+  </link>
   <joint name="base_link_joint" type="fixed">
-    <origin xyz="0 0 ${base_radius}" rpy="0 0 0" />
-    <parent link="base_footprint" />
-    <child link="base_link" />
+    <origin xyz="0 0 ${-(2*wheel_radius+base_height)}" rpy="0 0 0" />
+    <parent link="base_link" />
+    <child link="base_footprint" />
   </joint>
-  <xacro:wheel prefix="left" reflect="1" />
-  <xacro:wheel prefix="right" reflect="-1" />
-  <xacro:caster prefix="front" reflect="-1" />
-  <xacro:caster prefix="rear" reflect="1" />
+  <xacro:wheel prefix="left" y_reflect="1" />
+  <xacro:wheel prefix="right" y_reflect="-1" />
+  <xacro:caster prefix="front" x_reflect="1" />
+  <xacro:caster prefix="rear" x_reflect="-1" />
   <link name="laser_link">
     <visual>
@@ -52,14 +46,22 @@
     <xacro:cylinder_inertia m="${lidar_mass}" r="${lidar_radius}" h="${lidar_height}" />
   </link>
-  <joint name="hokuyo_joint" type="fixed">
+  <joint name="laser_joint" type="fixed">
     <origin xyz="0 0 ${base_height+lidar_radius/4}" rpy="0 0 0" />
     <parent link="base_link" />
     <child link="laser_link" />
   </joint>
-  <link name="imu"/>
+  <link name="imu">
+    <visual>
+      <origin xyz="0 0 0" rpy="0 0 0" />
+      <geometry>
+        <box size="0.02 0.02 0.001" />
+      </geometry>
+      <material name="red" />
+    </visual>
+  </link>
   <joint name="imu_joint" type="fixed">
-    <origin rpy="${pi} 0 0" xyz="-0.035.03 0.2"/>
+    <origin rpy="${pi} 0 0" xyz="-0.035 0.03 0.01" />
     <parent link="base_link" />
-    <child link="imu"/>
+    <child link="imu" />
   </joint>
   <!--

File: chefbot/chefbot_description/urdf/kbot_macros.xacro (robot description, xacro)
@@ -26,5 +26,5 @@
         </inertial>
     </xacro:macro>
-    <xacro:macro name="wheel" params="prefix reflect">
+    <xacro:macro name="wheel" params="prefix y_reflect">
         <link name="${prefix}_wheel_link">
             <visual>
@@ -47,6 +47,5 @@
             <parent link="base_link" />
             <child link="${prefix}_wheel_link" />
-            <origin xyz="0 ${reflect*(base_radius+base_wheel_gap)} 0" rpy="0 0 0" />
-            <joint_properties damping="1.0" friction="1.0" />
+            <origin xyz="0 ${y_reflect*(base_radius+wheel_yGap)} ${-wheel_zoff}" rpy="0 0 0" />
         </joint>
         <xacro:if value="${gazebo == 'true'}">
@@ -71,10 +70,9 @@
         </xacro:if>
     </xacro:macro>
-    <xacro:macro name="caster" params="prefix reflect">
-        <link name="${prefix}_caster_wheel">
+    <xacro:macro name="caster" params="prefix x_reflect">
+        <link name="${prefix}_caster">
             <visual>
-                <origin xyz="0 0 0" rpy="0 0 0" />
                 <geometry>
-                    <sphere radius="${caster_wheel_radius}" />
+                    <sphere radius="${caster_radius}" />
                 </geometry>
                 <material name="white" />
@@ -83,14 +81,14 @@
                 <origin xyz="0 0 0" rpy="0 0 0" />
                 <geometry>
-                    <sphere radius="${caster_wheel_radius}" />
+                    <sphere radius="${caster_radius}" />
                 </geometry>
             </collision>
-            <xacro:sphere_inertia m="${caster_wheel_mass}" r="${caster_wheel_radius}" />
+            <xacro:sphere_inertia m="${caster_mass}" r="${caster_radius}" />
         </link>
-        <joint name="${prefix}_caster_wheel_joint" type="fixed">
+        <joint name="${prefix}_caster_joint" type="fixed">
             <axis xyz="0 1 0" rpy="0 0 0" />
             <parent link="base_link" />
-            <child link="${prefix}_caster_wheel" />
-            <origin xyz="${reflect*caster_wheel_joint_offset} 0 -${caster_wheel_radius}" rpy="0 0 0" />
+            <child link="${prefix}_caster" />
+            <origin xyz="${x_reflect*caster_xoff} 0 -${caster_radius}" rpy="0 0 0" />
         </joint>
     </xacro:macro>

File: chefbot/chefbot_description/urdf/properties.xacro (robot description, xacro)
@@ -16,4 +16,6 @@
    Note: REP needs to be updated with the information below
    (currently in development and awaiting feedback)
+   This urdf is referred to:
+   https://navigation.ros.org/setup_guides/urdf/setup_urdf.html
 -->
   <xacro:property name="gazebo" value="true" />
@@ -37,6 +39,4 @@
   <xacro:property name="base_mass" value="4.0" /> <!-- in kg-->
   <xacro:property name="wheel_separation" value="${2*(wheel_radius+0.5*wheel_thick)" />
-  <xacro:property name="wheel_thick" value="0.01" />
-  <xacro:property name="base_wheel_gap" value="${base_radius*0.12}" />
   <xacro:property name='lidar_mass' value='0.125'/>
   <xacro:property name='lidar_radius' value='0.03'/>
@@ -44,12 +44,12 @@
   <!-- Wheels -->
   <xacro:property name="wheel_radius" value="0.035" />
+  <xacro:property name="wheel_thick" value="0.01" />
   <xacro:property name="wheel_mass" value="0.5" /> <!-- in kg-->
-  <xacro:property name="wheel_joint_offset" value="0.02" />
-  <xacro:property name="base_x_origin_to_wheel_origin" value="0.25" />
-  <xacro:property name="base_y_origin_to_wheel_origin" value="0.3" />
-  <xacro:property name="base_z_origin_to_wheel_origin" value="0.0" />
-  <xacro:property name="caster_wheel_radius" value="${wheel_radius*0.5}" />
-  <xacro:property name="caster_wheel_mass" value="0.1" />
-  <xacro:property name="caster_wheel_joint_offset" value="0.052" />
+  <xacro:property name="wheel_yGap" value="${base_radius*0.12}" />
+  <xacro:property name="wheel_zoff" value="${wheel_radius+base_height/2}"/>
+  <xacro:property name="wheel_xoff" value="0"/>
+  <xacro:property name="caster_xoff" value='${(base_radius-caster_radius)}'/>
+  <xacro:property name="caster_radius" value="${wheel_radius*0.5}" />
+  <xacro:property name="caster_mass" value="0.1" />
   <xacro:property name="cameraSize" value="0.05" />
   <xacro:property name="cameraMass" value="0.1" />

Commit message: refine xacro

File: chefbot/chefbot_description/urdf/kbot.xacro (robot description, xacro)
@@ -10,4 +10,12 @@
        add a simple link without inertia and make a joint between it and the chassis
     -->
+  <link name="base_footprint">
+    <xacro:box_inertia m="0" w="0" h="0" d="0" />
+  </link>
+  <joint name="base_footprint_joint" type="fixed">
+    <origin xyz="0 0 ${-(2*wheel_radius+base_height)}" rpy="0 0 0" />
+    <parent link="base_footprint" />
+    <child link="base_link" />
+  </joint>
   <link name="base_link">
     <visual>
@@ -24,16 +32,10 @@
     <xacro:cylinder_inertia m="${base_mass}" r="${base_radius}" h="${base_height}" />
   </link>
-  <link name="base_footprint">
-    <xacro:box_inertia m="0" w="0" h="0" d="0" />
-  </link>
-  <joint name="base_link_joint" type="fixed">
-    <origin xyz="0 0 ${-(2*wheel_radius+base_height)}" rpy="0 0 0" />
-    <parent link="base_link" />
-    <child link="base_footprint" />
-  </joint>
   <xacro:wheel prefix="left" y_reflect="1" />
   <xacro:wheel prefix="right" y_reflect="-1" />
   <xacro:caster prefix="front" x_reflect="1" />
+  <!-- it will be easy to know which direction is front in rviz
   <xacro:caster prefix="rear" x_reflect="-1" />
+  -->
   <link name="laser_link">
     <visual>
@@ -61,5 +63,5 @@
   </link>
   <joint name="imu_joint" type="fixed">
-    <origin rpy="${pi} 0 0" xyz="-0.035 0.03 0.01" />
+    <origin rpy="0 0 0" xyz="-0.035 0.03 0.01" />
     <parent link="base_link" />
     <child link="imu" />

File: chefbot/chefbot_description/urdf/kbot_macros.xacro (robot description, xacro)
@@ -44,4 +44,5 @@
         </link>
         <joint name="${prefix}_wheel_joint" type="continuous">
+            <!-- axis defines the rotation axis of the joint wrt the parent frame -->
             <axis xyz="0 1 0" rpy="0 0 0" />
             <parent link="base_link" />

File: chefbot/chefbot_description/urdf/properties.xacro (robot description, xacro)
@@ -54,3 +54,4 @@
   <xacro:property name="cameraSize" value="0.05" />
   <xacro:property name="cameraMass" value="0.1" />
+  <property name="DEG_TO_RAD" value="0.017453293" />
 </robot>

Commit message: fix xacro property w/o xacro: issue

File: chefbot/chefbot_description/urdf/kbot.xacro (robot description, xacro)
@@ -38,5 +38,5 @@
   <xacro:caster prefix="rear" x_reflect="-1" />
   -->
-  <link name="laser_link">
+  <link name="lidar_link">
     <visual>
       <origin xyz="0 0 0" rpy="0 0 0" />
@@ -48,8 +48,8 @@
     <xacro:cylinder_inertia m="${lidar_mass}" r="${lidar_radius}" h="${lidar_height}" />
   </link>
-  <joint name="laser_joint" type="fixed">
+  <joint name="lidar_joint" type="fixed">
     <origin xyz="0 0 ${base_height+lidar_radius/4}" rpy="0 0 0" />
     <parent link="base_link" />
-    <child link="laser_link" />
+    <child link="lidar_link" />
   </joint>
   <link name="imu">
@@ -59,5 +59,5 @@
         <box size="0.02 0.02 0.001" />
       </geometry>
-      <material name="red" />
+      <material name="green" />
     </visual>
   </link>
@@ -68,5 +68,5 @@
   </joint>
   <!--
-    <link name="camera">
+    <link name="camera_link">
       <collision>
         <origin xyz="0 0 0" rpy="0 0 0"/>

File: chefbot/chefbot_description/urdf/materials.xacro (robot description, xacro)
@@ -3,4 +3,7 @@
     <material name="green">
         <color rgba="0.0 1.0 0.0 1.0" />
+    </material>
+    <material name="dark green">
+        <color rgba="0 86 69 1.0" />
     </material>
     <material name="grey">

File: chefbot/chefbot_description/urdf/properties.xacro (robot description, xacro)
@@ -54,4 +54,4 @@
   <xacro:property name="cameraSize" value="0.05" />
   <xacro:property name="cameraMass" value="0.1" />
-  <property name="DEG_TO_RAD" value="0.017453293" />
+  <xacro:property name="DEG_TO_RAD" value="0.017453293" />
 </robot>

Commit message: add udev rules for usb devices

File: chefbot/chefbot_description/urdf/kbot.xacro (robot description, xacro)
@@ -11,13 +11,15 @@
     -->
   <link name="base_footprint">
-    <xacro:box_inertia m="0" w="0" h="0" d="0" />
+    <xacro:box_inertia m="0.001" w="0.001" h="0.001" d="0.001" />
+    <visual>
+      <origin xyz="0 0 0" rpy="0 0 0" />
+      <geometry>
+          <box size="0.001 0.001 0.001" />
+      </geometry>
+  </visual>
   </link>
-  <joint name="base_footprint_joint" type="fixed">
-    <origin xyz="0 0 ${-(2*wheel_radius+base_height)}" rpy="0 0 0" />
-    <parent link="base_footprint" />
-    <child link="base_link" />
-  </joint>
   <link name="base_link">
     <visual>
+      <origin xyz="0 0 0" rpy="0 0 0" />
       <geometry>
         <cylinder radius="${base_radius}" length="${base_height}" />
@@ -26,4 +28,5 @@
     </visual>
     <collision>
+      <origin xyz="0 0 0" rpy="0 0 0 " />
       <geometry>
         <cylinder radius="${base_radius}" length="${base_height}" />
@@ -32,4 +35,9 @@
     <xacro:cylinder_inertia m="${base_mass}" r="${base_radius}" h="${base_height}" />
   </link>
+  <joint name="base_link_joint" type="fixed">
+    <origin xyz="0 0 ${(2*wheel_radius)}" rpy="0 0 0" />
+    <parent link="base_footprint" />
+    <child link="base_link" />
+  </joint>
   <xacro:wheel prefix="left" y_reflect="1" />
   <xacro:wheel prefix="right" y_reflect="-1" />
@@ -49,5 +57,5 @@
   </link>
   <joint name="lidar_joint" type="fixed">
-    <origin xyz="0 0 ${base_height+lidar_radius/4}" rpy="0 0 0" />
+    <origin xyz="0 0 ${15*base_height+lidar_radius/4}" rpy="0 0 0" />
     <parent link="base_link" />
     <child link="lidar_link" />

File: chefbot/chefbot_description/urdf/properties.xacro (robot description, xacro)
@@ -51,5 +51,5 @@
   <xacro:property name="caster_xoff" value='${(base_radius-caster_radius)}'/>
   <xacro:property name="caster_radius" value="${wheel_radius*0.5}" />
-  <xacro:property name="caster_mass" value="0.1" />
+  <xacro:property name="caster_mass" value="0.2" />
   <xacro:property name="cameraSize" value="0.05" />
   <xacro:property name="cameraMass" value="0.1" />

Commit message: tune nav but not working

File: chefbot/chefbot_description/urdf/kbot.xacro (robot description, xacro)
@@ -11,4 +11,5 @@
     -->
   <link name="base_footprint">
+    <!--
     <xacro:box_inertia m="0.001" w="0.001" h="0.001" d="0.001" />
     <visual>
@@ -18,4 +19,5 @@
       </geometry>
   </visual>
+    -->
   </link>
   <link name="base_link">
@@ -61,5 +63,5 @@
     <child link="lidar_link" />
   </joint>
-  <link name="imu">
+  <link name="imu_link">
     <visual>
       <origin xyz="0 0 0" rpy="0 0 0" />
@@ -73,5 +75,5 @@
     <origin rpy="0 0 0" xyz="-0.035 0.03 0.01" />
     <parent link="base_link" />
-    <child link="imu" />
+    <child link="imu_link" />
   </joint>
   <!--

Commit message: nav works by using turtlebot3's param

File: chefbot/chefbot_description/urdf/kbot.xacro (robot description, xacro)
@@ -56,8 +56,7 @@
       <material name="blue" />
     </visual>
-    <xacro:cylinder_inertia m="${lidar_mass}" r="${lidar_radius}" h="${lidar_height}" />
   </link>
   <joint name="lidar_joint" type="fixed">
-    <origin xyz="0 0 ${15*base_height+lidar_radius/4}" rpy="0 0 0" />
+   <origin xyz="0 0 ${3.1*2*wheel_radius}" rpy="0 0 0" />
     <parent link="base_link" />
     <child link="lidar_link" />

Commit message: add camrea in urdf

File: chefbot/chefbot_description/urdf/kbot.xacro (robot description, xacro)
@@ -11,14 +11,17 @@
     -->
   <link name="base_footprint">
-    <!--
     <xacro:box_inertia m="0.001" w="0.001" h="0.001" d="0.001" />
     <visual>
       <origin xyz="0 0 0" rpy="0 0 0" />
       <geometry>
-          <box size="0.001 0.001 0.001" />
+        <box size="0.001 0.001 0.001" />
       </geometry>
-  </visual>
-    -->
+    </visual>
   </link>
+  <joint name="base_footprint_joint" type="fixed">
+    <origin rpy="0 0 0" xyz="0 0 0.04" />
+    <parent link="base_footprint" />
+    <child link="base_link" />
+  </joint>
   <link name="base_link">
     <visual>
@@ -58,5 +61,5 @@
   </link>
   <joint name="lidar_joint" type="fixed">
-   <origin xyz="0 0 ${3.1*2*wheel_radius}" rpy="0 0 0" />
+    <origin xyz="0 0 ${3.1*2*wheel_radius}" rpy="0 0 0" />
     <parent link="base_link" />
     <child link="lidar_link" />
@@ -76,21 +79,25 @@
     <child link="imu_link" />
   </joint>
-  <!--
-    <link name="camera_link">
-      <collision>
-        <origin xyz="0 0 0" rpy="0 0 0"/>
-        <geometry>
-          <box size="${cameraSize} ${cameraSize} ${cameraSize}"/>
-        </geometry>
-      </collision>
-      <visual>
-        <origin xyz="0 0 0" rpy="0 0 0"/>
-        <geometry>
-          <box size="${cameraSize} ${cameraSize} ${cameraSize}"/>
-        </geometry>
-        <material name="blue"/>
-      </visual>
-      <xacro:box_inertia m="${cameraMass}" w="${cameraSize}" h="${cameraSize}" d="${cameraSize}" />
-    </link>
-  -->
+  <link name="camera_link">
+    <collision>
+      <origin xyz="0 0 0" rpy="0 0 0" />
+      <geometry>
+        <box size="${cameraSize} ${cameraSize} ${cameraSize}" />
+      </geometry>
+    </collision>
+    <visual>
+      <origin xyz="0 0 0" rpy="0 0 0" />
+      <geometry>
+        <box size="${cameraSize} ${cameraSize} ${cameraSize}" />
+      </geometry>
+      <material name="red" />
+    </visual>
+    <xacro:box_inertia m="${cameraMass}" w="${cameraSize}" h="${cameraSize}" d="${cameraSize}" />
+  </link>
+  <joint name="camera_joint" type="fixed">
+    <parent link="base_link" />
+    <child link="camera_link" />
+    <origin rpy="0 0 0" xyz="0.09 0.0 0.12" />
+    <axis xyz="1 0 0" />
+  </joint>
 </robot>

File: chefbot/chefbot_description/urdf/properties.xacro (robot description, xacro)
@@ -52,5 +52,5 @@
   <xacro:property name="caster_radius" value="${wheel_radius*0.5}" />
   <xacro:property name="caster_mass" value="0.2" />
-  <xacro:property name="cameraSize" value="0.05" />
-  <xacro:property name="cameraMass" value="0.1" />
+  <xacro:property name="cameraSize" value="0.04" />
+  <xacro:property name="cameraMass" value="0.01" />
 </robot>
