Commit message: incl ekf in nav.launch, tf2, /dev/arduino, move_base1

File: chefbot/chefbot_description/urdf/kbot_macros.xacro (robot description, xacro)
@@ -29,5 +29,5 @@
         <link name="${prefix}_wheel_link">
             <visual>
-                <origin xyz="0 0 0" rpy="${M_PI_2} 0 0" />
+                <!-- <origin xyz="0 0 0" rpy="${M_PI_2} 0 0" /> -->
                 <geometry>
                     <cylinder radius="${wheel_radius}" length="${wheel_thick}" />
@@ -36,5 +36,5 @@
             </visual>
             <collision>
-                <origin xyz="0 0 0 " rpy="${M_PI_2} 0 0" />
+                <!-- <origin xyz="0 0 0 " rpy="${M_PI_2} 0 0" /> -->
                 <geometry>
                     <cylinder radius="${wheel_radius}" length="${wheel_thick}" />
@@ -45,8 +45,8 @@
         <joint name="${prefix}_wheel_joint" type="continuous">
             <!-- axis defines the rotation axis of the joint wrt the parent frame -->
-            <axis xyz="0 1 0" rpy="0 0 0" />
+            <axis xyz="0 0 1" rpy="0 0 0" />
             <parent link="base_link" />
             <child link="${prefix}_wheel_link" />
-            <origin xyz="0 ${y_reflect*(base_radius+wheel_yGap)} ${-wheel_zoff}" rpy="0 0 0" />
+            <origin xyz="0 ${y_reflect*(base_radius+wheel_yGap)} ${-wheel_zoff}" rpy="${M_PI_2} 0 0" />
         </joint>
         <xacro:if value="${gazebo == 'true'}">
@@ -80,5 +80,4 @@
             </visual>
             <collision>
-                <origin xyz="0 0 0" rpy="0 0 0" />
                 <geometry>
                     <sphere radius="${caster_radius}" />
@@ -88,5 +87,5 @@
         </link>
         <joint name="${prefix}_caster_joint" type="fixed">
-            <axis xyz="0 1 0" rpy="0 0 0" />
+            <axis xyz="0 0 1" rpy="0 0 0" />
             <parent link="base_link" />
             <child link="${prefix}_caster" />

Commit message: add wheel mesh file for urdf

File: chefbot/chefbot_description/urdf/kbot_macros.xacro (robot description, xacro)
@@ -31,5 +31,6 @@
                 <!-- <origin xyz="0 0 0" rpy="${M_PI_2} 0 0" /> -->
                 <geometry>
-                    <cylinder radius="${wheel_radius}" length="${wheel_thick}" />
+                    <!-- <cylinder radius="${wheel_radius}" length="${wheel_thick}" />  -->
+                    <mesh filename="package://urdf_tutorial/meshes/wheel.dae"/>
                 </geometry>
                 <material name="black" />
@@ -39,4 +40,5 @@
                 <geometry>
                     <cylinder radius="${wheel_radius}" length="${wheel_thick}" />
+                    <!-- <mesh filename="package:://chefbot_description/meshes/piCamera.stl" scale="0.005 0.005 0.005"/>-->
                 </geometry>
             </collision>

File: chefbot/chefbot_description/urdf/wheel.urdf.xacro (robot description, xacro)
@@ -13,5 +13,6 @@
         <origin xyz="0 0 0" rpy="${flipY*M_PI/2} 0  0 " />
         <geometry>
-          <cylinder length="${wheel_height}" radius="${wheel_radius}" />
+          <!-- <cylinder length="${wheel_height}" radius="${wheel_radius}" /> -->
+          <mesh filename="package:://chefbot_description/meshes/wheel.dae"/>
         </geometry>
         <material name="DarkGray" />
@@ -20,5 +21,8 @@
         <origin xyz="0 0 0" rpy="${flipY*M_PI/2} 0 0 " />
         <geometry>
+          <!--
           <cylinder length="${wheel_height}" radius="${wheel_radius}" />
+          -->
+          <mesh filename="package:://chefbot_description/meshes/wheel.dae"/>
         </geometry>
       </collision>

Commit message: add udev rules

File: chefbot/chefbot_description/urdf/kbot_macros.xacro (robot description, xacro)
@@ -77,5 +77,6 @@
             <visual>
                 <geometry>
-                    <sphere radius="${caster_radius}" />
+                    <!-- <sphere radius="${caster_radius}" /> -->
+                    <mesh filename="package://urdf_tutorial/meshes/caster_wheel.stl" scale='0.8 0.8 0.8'/>
                 </geometry>
                 <material name="white" />
@@ -92,5 +93,6 @@
             <parent link="base_link" />
             <child link="${prefix}_caster" />
-            <origin xyz="${x_reflect*caster_xoff} 0 -${caster_radius}" rpy="0 0 0" />
+            <!-- <origin xyz="${x_reflect*caster_xoff} 0 -${caster_radius}" rpy="0 0 0" /> -->
+            <origin xyz="${x_reflect*caster_xoff} 0 0" rpy="-1.571 0 1.571" />
         </joint>
     </xacro:macro>
