Commit message: add gitignore extn

File: chefbot/chefbot_description/urdf/diff_wheeled_robot.urdf (robot description, URDF)
Before this commit: robot differential_wheeled_robot, 6 links, 5 joints
Joints:
- joint caster_back_joint: origin xyz=-0.135 0.0 0.009 rpy=-1.57079632679 0 0 -> xyz=-0.135 0.0 0.009 rpy=-1.5707963267948966 0 0
- joint caster_front_joint: origin xyz=0.115 0.0 0.007 rpy=-1.57079632679 0 0 -> xyz=0.115 0.0 0.007 rpy=-1.5707963267948966 0 0
- joint front_left_wheel_joint: origin xyz=0.0 0.15 0.0 rpy=0 0 0 -> xyz=0.0 -0.15 0.0 rpy=0 0 0
- joint front_right_wheel_joint: origin xyz=0.0 -0.15 0.0 rpy=0 0 0 -> xyz=0.0 0.15 0.0 rpy=0 0 0

File: chefbot/chefbot_description/urdf/diff_wheeled_robot.xacro (robot description, xacro)
@@ -1,17 +1,17 @@
 <?xml version="1.0"?>
 <robot name="differential_wheeled_robot" xmlns:xacro="http://ros.org/wiki/xacro">
-  <xacro:include filename="$(find chefbot_description)/urdf/wheel.urdf.xacro" />
-  <!-- Defining the colors used in this robot -->
+  <xacro:include filename="$(find mastering_ros_robot_description_pkg)/urdf/wheel.urdf.xacro" />
+<!-- Defining the colors used in this robot -->
   <material name="Black">
-    <color rgba="0.0 0.0 0.0 1.0" />
+    <color rgba="0.0 0.0 0.0 1.0"/>
   </material>
   <material name="Red">
-    <color rgba="0.8 0.0 0.0 1.0" />
+    <color rgba="0.8 0.0 0.0 1.0"/>
   </material>
   <material name="White">
-    <color rgba="1.0 1.0 1.0 1.0" />
+    <color rgba="1.0 1.0 1.0 1.0"/>
   </material>
   <material name="Blue">
-    <color rgba="0.0 0.0 0.8 1.0" />
+    <color rgba="0.0 0.0 0.8 1.0"/>
   </material>
   <!-- PROPERTY LIST -->
@@ -36,6 +36,5 @@
   <xacro:property name="caster_b_mass" value="0.5" /> <!-- in kg-->
   <!-- Wheels -->
-  <xacro:property name="wheel_mass" value="2.5" />
-  --> <!-- in kg-->
+  <xacro:property name="wheel_mass" value="2.5" /> --> <!-- in kg-->
   <xacro:property name="base_x_origin_to_wheel_origin" value="0.25" />
   <xacro:property name="base_y_origin_to_wheel_origin" value="0.3" />
@@ -45,5 +44,7 @@
   <!-- Macro for calculating inertia of cylinder -->
   <xacro:macro name="cylinder_inertia" params="m r h">
-    <inertia ixx="${m*(3*r*r+h*h)/12}" ixy="0" ixz="0" iyy="${m*(3*r*r+h*h)/12}" iyz="0" izz="${m*r*r/2}" />
+    <inertia  ixx="${m*(3*r*r+h*h)/12}" ixy = "0" ixz = "0"
+              iyy="${m*(3*r*r+h*h)/12}" iyz = "0"
+              izz="${m*r*r/2}" />
   </xacro:macro>
   <!-- BASE-FOOTPRINT -->
@@ -53,11 +54,13 @@
       <mass value="0.0001" />
       <origin xyz="0 0 0" />
-      <inertia ixx="0.0001" ixy="0.0" ixz="0.0" iyy="0.0001" iyz="0.0" izz="0.0001" />
+      <inertia ixx="0.0001" ixy="0.0" ixz="0.0"
+          iyy="0.0001" iyz="0.0"
+          izz="0.0001" />
     </inertial>
     <visual>
-      <origin xyz="0 0 0" rpy="0 0 0" />
-      <geometry>
-        <box size="0.001 0.001 0.001" />
-      </geometry>
+        <origin xyz="0 0 0" rpy="0 0 0" />
+        <geometry>
+            <box size="0.001 0.001 0.001" />
+        </geometry>
     </visual>
   </link>
@@ -67,5 +70,5 @@
   <joint name="base_footprint_joint" type="fixed">
     <origin xyz="0 0 ${wheel_radius - base_z_origin_to_wheel_origin}" rpy="0 0 0" />
-    <parent link="base_footprint" />
+    <parent link="base_footprint"/>
     <child link="base_link" />
   </joint>
@@ -74,11 +77,13 @@
       <mass value="${base_mass}" />
       <origin xyz="0 0 0" />
-      <inertia ixx="0.0001" ixy="0.0" ixz="0.0" iyy="0.0001" iyz="0.0" izz="0.0001" />
-      <cylinder_inertia m="${base_mass}" r="${base_radius}" h="${base_height}" />
+      <inertia ixx="0.0001" ixy="0.0" ixz="0.0"
+          iyy="0.0001" iyz="0.0"
+          izz="0.0001" />
+      <cylinder_inertia  m="${base_mass}" r="${base_radius}" h="${base_height}" />
     </inertial>
     <visual>
       <origin xyz="0 0 0" rpy="0 0 0" />
       <geometry>
-        <cylinder length="${base_height}" radius="${base_radius}" />
+          <cylinder length="${base_height}" radius="${base_radius}" />
       </geometry>
       <material name="White" />
@@ -87,5 +92,5 @@
       <origin xyz="0 0 0" rpy="0 0 0 " />
       <geometry>
-        <cylinder length="${base_height}" radius="${base_radius}" />
+          <cylinder length="${base_height}" radius="${base_radius}" />
       </geometry>
     </collision>
@@ -99,5 +104,5 @@
       <origin xyz="0 0.02 0" rpy="${M_PI/2} 0 0" />
       <geometry>
-        <sphere radius="${caster_f_radius}" />
+				<sphere radius="${caster_f_radius}" />
       </geometry>
       <material name="Black" />
@@ -105,18 +110,20 @@
     <collision>
       <geometry>
-        <sphere radius="${caster_f_radius}" />
+				<sphere radius="${caster_f_radius}" />
       </geometry>
-      <origin xyz="0 0.02 0" rpy="${M_PI/2} 0 0" />
+    <origin xyz="0 0.02 0" rpy="${M_PI/2} 0 0" />
     </collision>
     <inertial>
       <mass value="${caster_f_mass}" />
       <origin xyz="0 0 0" />
-      <inertia ixx="0.001" ixy="0.0" ixz="0.0" iyy="0.001" iyz="0.0" izz="0.001" />
+      <inertia ixx="0.001" ixy="0.0" ixz="0.0"
+               iyy="0.001" iyz="0.0"
+               izz="0.001" />
     </inertial>
   </link>
-  <joint name="caster_front_joint" type="fixed">
-    <parent link="base_link" />
-    <child link="caster_front_link" />
-    <origin xyz="0.115 0.0 0.007" rpy="${-M_PI/2} 0 0" />
+	<joint name="caster_front_joint" type="fixed">
+    <parent link="base_link"/>
+    <child link="caster_front_link"/>
+    <origin xyz="0.115 0.0 0.007" rpy="${-M_PI/2} 0 0"/>
   </joint>
   <gazebo reference="caster_front_link">
@@ -124,55 +131,57 @@
   </gazebo>
   <link name="caster_back_link">
-    <visual>
-      <origin xyz="0.02 0.02 0 " rpy="${M_PI/2} 0 0" />
-      <geometry>
-        <sphere radius="${caster_b_radius}" />
-      </geometry>
-      <material name="Black" />
-    </visual>
-    <collision>
-      <geometry>
-        <sphere radius="${caster_b_radius}" />
-      </geometry>
-      <origin xyz="0 0.02 0 " rpy="${M_PI/2} 0 0" />
+  <visual>
+    <origin xyz="0.02 0.02 0 " rpy="${M_PI/2} 0 0" />
+    <geometry>
+			<sphere radius="${caster_b_radius}" />
+    </geometry>
+    <material name="Black" />
+  </visual>
+  <collision>
+    <geometry>
+			<sphere radius="${caster_b_radius}" />
+     </geometry>
+     <origin xyz="0 0.02 0 " rpy="${M_PI/2} 0 0" />
     </collision>
     <inertial>
       <mass value="${caster_b_mass}" />
       <origin xyz="0 0 0" />
-      <inertia ixx="0.001" ixy="0.0" ixz="0.0" iyy="0.001" iyz="0.0" izz="0.001" />
+      <inertia ixx="0.001" ixy="0.0" ixz="0.0"
+               iyy="0.001" iyz="0.0"
+               izz="0.001" />
     </inertial>
   </link>
   <joint name="caster_back_joint" type="fixed">
-    <parent link="base_link" />
-    <child link="caster_back_link" />
-    <origin xyz="-0.135 0.0 0.009" rpy="${-M_PI/2} 0 0" />
+    <parent link="base_link"/>
+    <child link="caster_back_link"/>
+    <origin xyz="-0.135 0.0 0.009" rpy="${-M_PI/2} 0 0"/>
   </joint>
   <gazebo reference="caster_back_link">
-    <turnGravityOff>false</turnGravityOff>
+   <turnGravityOff>false</turnGravityOff>
   </gazebo>
-  <xacro:wheel fb="front" lr="right" parent="base_link" translateX="0" translateY="-0.5" flipY="1" />
-  <xacro:wheel fb="front" lr="left" parent="base_link" translateX="0" translateY="0.5" flipY="1" />
-  <gazebo>
-    <plugin name="differential_drive_controller" filename="libgazebo_ros_diff_drive.so">
-      <legacyMode>true</legacyMode>
-      <rosDebugLevel>Debug</rosDebugLevel>
-      <publishWheelTF>false</publishWheelTF>
-      <robotNamespace>/</robotNamespace>
-      <publishTf>1</publishTf>
-      <publishWheelJointState>false</publishWheelJointState>
-      <alwaysOn>true</alwaysOn>
-      <updateRate>100.0</updateRate>
-      <leftJoint>front_left_wheel_joint</leftJoint>
-      <rightJoint>front_right_wheel_joint</rightJoint>
-      <wheelSeparation>${2*base_radius}</wheelSeparation>
-      <wheelDiameter>${2*wheel_radius}</wheelDiameter>
-      <broadcastTF>1</broadcastTF>
-      <wheelTorque>30</wheelTorque>
-      <wheelAcceleration>1.8</wheelAcceleration>
-      <commandTopic>cmd_vel</commandTopic>
-      <odometryFrame>odom</odometryFrame>
-      <odometryTopic>odom</odometryTopic>
-      <robotBaseFrame>base_footprint</robotBaseFrame>
-    </plugin>
+  <xacro:wheel fb="front" lr="right" parent="base_link" translateX="0" translateY="-0.5" flipY="1"/>
+	<xacro:wheel fb="front" lr="left" parent="base_link" translateX="0" translateY="0.5" flipY="1"/>
+	<gazebo>
+  	<plugin name="differential_drive_controller" filename="libgazebo_ros_diff_drive.so">
+	    <legacyMode>true</legacyMode>
+	    <rosDebugLevel>Debug</rosDebugLevel>
+	    <publishWheelTF>false</publishWheelTF>
+	    <robotNamespace>/</robotNamespace>
+	    <publishTf>1</publishTf>
+	    <publishWheelJointState>false</publishWheelJointState>
+	    <alwaysOn>true</alwaysOn>
+	    <updateRate>100.0</updateRate>
+	    <leftJoint>front_left_wheel_joint</leftJoint>
+	    <rightJoint>front_right_wheel_joint</rightJoint>
+	    <wheelSeparation>${2*base_radius}</wheelSeparation>
+	    <wheelDiameter>${2*wheel_radius}</wheelDiameter>
+	    <broadcastTF>1</broadcastTF>
+	    <wheelTorque>30</wheelTorque>
+	    <wheelAcceleration>1.8</wheelAcceleration>
+	    <commandTopic>cmd_vel</commandTopic>
+	    <odometryFrame>odom</odometryFrame>
+	    <odometryTopic>odom</odometryTopic>
+	    <robotBaseFrame>base_footprint</robotBaseFrame>
+   </plugin>
   </gazebo>
 </robot>

File: chefbot/chefbot_description/urdf/diff_wheeled_robot_with_laser.xacro (robot description, xacro)
@@ -1,5 +1,5 @@
 <?xml version="1.0"?>
 <robot name="differential_wheeled_robot" xmlns:xacro="http://ros.org/wiki/xacro">
-  <xacro:include filename="$(find chefbot_description)/urdf/wheel.urdf.xacro" />
+  <xacro:include filename="$(find mastering_ros_robot_description_pkg)/urdf/wheel.urdf.xacro" />
 	<!-- Defining the colors used in this robot -->
   <material name="Black">

File: chefbot/chefbot_description/urdf/kbot.xacro (robot description, xacro)
@@ -4,24 +4,23 @@
   <xacro:include filename="$(find chefbot_description)/urdf/materials.xacro" />
   <xacro:include filename="$(find chefbot_description)/urdf/kbot_macros.xacro" />
+  <!--
   <xacro:if value="${gazebo == 'true'}">
     <xacro:include filename="$(find chefbot_description)/urdf/kbot.gazebo" />
   </xacro:if>
+-->
   <!-- The physic engine does not accept a base_link with inertia. It is then useful to
        add a simple link without inertia and make a joint between it and the chassis
     -->
   <link name="base_footprint">
+    <!--
     <xacro:box_inertia m="0.001" w="0.001" h="0.001" d="0.001" />
     <visual>
       <origin xyz="0 0 0" rpy="0 0 0" />
       <geometry>
-        <box size="0.001 0.001 0.001" />
+          <box size="0.001 0.001 0.001" />
       </geometry>
-    </visual>
+  </visual>
+    -->
   </link>
-  <joint name="base_footprint_joint" type="fixed">
-    <origin rpy="0 0 0" xyz="0 0 0.04" />
-    <parent link="base_footprint" />
-    <child link="base_link" />
-  </joint>
   <link name="base_link">
     <visual>
@@ -61,5 +60,5 @@
   </link>
   <joint name="lidar_joint" type="fixed">
-    <origin xyz="0 0 ${3.1*2*wheel_radius}" rpy="0 0 0" />
+   <origin xyz="0 0 ${3.1*2*wheel_radius}" rpy="0 0 0" />
     <parent link="base_link" />
     <child link="lidar_link" />
@@ -79,25 +78,21 @@
     <child link="imu_link" />
   </joint>
-  <link name="camera_link">
-    <collision>
-      <origin xyz="0 0 0" rpy="0 0 0" />
-      <geometry>
-        <box size="${cameraSize} ${cameraSize} ${cameraSize}" />
-      </geometry>
-    </collision>
-    <visual>
-      <origin xyz="0 0 0" rpy="0 0 0" />
-      <geometry>
-        <box size="${cameraSize} ${cameraSize} ${cameraSize}" />
-      </geometry>
-      <material name="red" />
-    </visual>
-    <xacro:box_inertia m="${cameraMass}" w="${cameraSize}" h="${cameraSize}" d="${cameraSize}" />
-  </link>
-  <joint name="camera_joint" type="fixed">
-    <parent link="base_link" />
-    <child link="camera_link" />
-    <origin rpy="0 0 0" xyz="0.09 0.0 0.12" />
-    <axis xyz="1 0 0" />
-  </joint>
+  <!--
+    <link name="camera_link">
+      <collision>
+        <origin xyz="0 0 0" rpy="0 0 0"/>
+        <geometry>
+          <box size="${cameraSize} ${cameraSize} ${cameraSize}"/>
+        </geometry>
+      </collision>
+      <visual>
+        <origin xyz="0 0 0" rpy="0 0 0"/>
+        <geometry>
+          <box size="${cameraSize} ${cameraSize} ${cameraSize}"/>
+        </geometry>
+        <material name="blue"/>
+      </visual>
+      <xacro:box_inertia m="${cameraMass}" w="${cameraSize}" h="${cameraSize}" d="${cameraSize}" />
+    </link>
+  -->
 </robot>

File: chefbot/chefbot_description/urdf/kbot_macros.xacro (robot description, xacro)
@@ -1,4 +1,4 @@
 <?xml version="1.0"?>
-<robot xmlns:xacro="http://www.ros.org/wiki/xacro" name="roachbot">
+<robot xmlns:xacro="http://www.ros.org/wiki/xacro">
     <xacro:macro name="default_inertial" params="z_value i_value mass">
         <inertial>
@@ -29,16 +29,14 @@
         <link name="${prefix}_wheel_link">
             <visual>
-                <!-- <origin xyz="0 0 0" rpy="${M_PI_2} 0 0" /> -->
+                <!-- <origin xyz="0 0 0" rpy="${M_PI_2} 0 0" -->
                 <geometry>
-                    <!-- <cylinder radius="${wheel_radius}" length="${wheel_thick}" />  -->
-                    <mesh filename="package://urdf_tutorial/meshes/wheel.dae"/>
+                    <cylinder radius="${wheel_radius}" length="${wheel_thick}" />
                 </geometry>
                 <material name="black" />
             </visual>
             <collision>
-                <!-- <origin xyz="0 0 0 " rpy="${M_PI_2} 0 0" /> -->
+                <!-- <origin xyz="0 0 0 " rpy="${M_PI_2} 0 0" -->
                 <geometry>
                     <cylinder radius="${wheel_radius}" length="${wheel_thick}" />
-                    <!-- <mesh filename="package:://chefbot_description/meshes/piCamera.stl" scale="0.005 0.005 0.005"/>-->
                 </geometry>
             </collision>
@@ -52,24 +50,4 @@
             <origin xyz="0 ${y_reflect*(base_radius+wheel_yGap)} ${-wheel_zoff}" rpy="${M_PI_2} 0 0" />
         </joint>
-        <xacro:if value="${gazebo == 'true'}">
-            <gazebo reference="${prefix}_wheel_link">
-                <mu1 value="1.0" />
-                <mu2 value="1.0" />
-                <kp value="10000000.0" />
-                <kd value="0.0" />
-                <fdir1 value="1 0 0" />
-                <material>Gazebo/FlatBlack</material>
-            </gazebo>
-            <transmission name="${prefix}_trans">
-                <type>transmission_interface/SimpleTransmission</type>
-                <joint name="${prefix}_wheel_joint">
-                    <hardwareInterface>hardware_interface/EffortJointInterface</hardwareInterface>
-                </joint>
-                <actuator name="${prefix}Motor">
-                    <hardwareInterface>hardware_interface/EffortJointInterface</hardwareInterface>
-                    <mechanicalReduction>1</mechanicalReduction>
-                </actuator>
-            </transmission>
-        </xacro:if>
     </xacro:macro>
     <xacro:macro name="caster" params="prefix x_reflect">
@@ -77,6 +55,5 @@
             <visual>
                 <geometry>
-                    <!-- <sphere radius="${caster_radius}" /> -->
-                    <mesh filename="package://urdf_tutorial/meshes/caster_wheel.stl" scale='0.8 0.8 0.8'/>
+                    <sphere radius="${caster_radius}" />
                 </geometry>
                 <material name="white" />
@@ -93,9 +70,9 @@
             <parent link="base_link" />
             <child link="${prefix}_caster" />
-            <!-- <origin xyz="${x_reflect*caster_xoff} 0 -${caster_radius}" rpy="0 0 0" /> -->
-            <origin xyz="${x_reflect*caster_xoff} 0 0" rpy="-1.571 0 1.571" />
+            <origin xyz="${x_reflect*caster_xoff} 0 -${caster_radius}" rpy="0 0 0" />
         </joint>
     </xacro:macro>
-    <!--
+</robot>
+<!--
     <xacro:macro name="joint_wheel" params="name child parent origin_xyz">
         <joint name="${name}" type="continuous">
@@ -109,5 +86,5 @@
     </xacro:macro>
 -->
-    <!--
+<!--
     <xacro:macro name="link_wheel" params="lr flipY">
         <link name="${lr}_wheel_link">
@@ -129,3 +106,2 @@
     </xacro:macro>
 -->
-</robot>

File: chefbot/chefbot_description/urdf/materials.xacro (robot description, xacro)
@@ -1,4 +1,4 @@
 <?xml version="1.0"?>
-<robot xmlns:xacro="http://www.ros.org/wiki/xacro" name="roachbot">
+<robot xmlns:xacro="http://www.ros.org/wiki/xacro" >
     <material name="green">
         <color rgba="0.0 1.0 0.0 1.0" />

File: chefbot/chefbot_description/urdf/properties.xacro (robot description, xacro)
@@ -1,4 +1,4 @@
 <?xml version="1.0"?>
-<robot xmlns:xacro="http://ros.org/wiki/xacro" name="roachbot">
+<robot xmlns:xacro="http://ros.org/wiki/xacro">
   <!--
   These properties must be observed by any machine
@@ -19,5 +19,5 @@
    https://navigation.ros.org/setup_guides/urdf/setup_urdf.html
 -->
-  <xacro:property name="gazebo" value="true" />
+  <xacro:property name="gazebo" value="false" />
   <xacro:property name="hokuyo_size" value="0.03" />
   <xacro:property name="cam_px" value="-0.087" />
@@ -39,7 +39,7 @@
   <xacro:property name="base_mass" value="4.0" /> <!-- in kg-->
   <xacro:property name="wheel_separation" value="${2*(wheel_radius+0.5*wheel_thick)" />
-  <xacro:property name='lidar_mass' value='0.125'/>
-  <xacro:property name='lidar_radius' value='0.03'/>
-  <xacro:property name='lidar_height' value='0.04'/>
+  <xacro:property name='lidar_mass' value='0.125' />
+  <xacro:property name='lidar_radius' value='0.03' />
+  <xacro:property name='lidar_height' value='0.04' />
   <!-- Wheels -->
   <xacro:property name="wheel_radius" value="0.034" />
@@ -47,7 +47,7 @@
   <xacro:property name="wheel_mass" value="0.5" /> <!-- in kg-->
   <xacro:property name="wheel_yGap" value="${base_radius*0.12}" />
-  <xacro:property name="wheel_zoff" value="${wheel_radius+base_height/2}"/>
-  <xacro:property name="wheel_xoff" value="0"/>
-  <xacro:property name="caster_xoff" value='${(base_radius-caster_radius)}'/>
+  <xacro:property name="wheel_zoff" value="${wheel_radius+base_height/2}" />
+  <xacro:property name="wheel_xoff" value="0" />
+  <xacro:property name="caster_xoff" value='${(base_radius-caster_radius)}' />
   <xacro:property name="caster_radius" value="${wheel_radius*0.5}" />
   <xacro:property name="caster_mass" value="0.2" />

File: chefbot/chefbot_description/urdf/wheel.urdf.xacro (robot description, xacro)
@@ -13,6 +13,5 @@
         <origin xyz="0 0 0" rpy="${flipY*M_PI/2} 0  0 " />
         <geometry>
-          <!-- <cylinder length="${wheel_height}" radius="${wheel_radius}" /> -->
-          <mesh filename="package:://chefbot_description/meshes/wheel.dae"/>
+          <cylinder length="${wheel_height}" radius="${wheel_radius}" />
         </geometry>
         <material name="DarkGray" />
@@ -21,8 +20,5 @@
         <origin xyz="0 0 0" rpy="${flipY*M_PI/2} 0 0 " />
         <geometry>
-          <!--
           <cylinder length="${wheel_height}" radius="${wheel_radius}" />
-          -->
-          <mesh filename="package:://chefbot_description/meshes/wheel.dae"/>
         </geometry>
       </collision>
@@ -58,5 +54,5 @@
       <actuator name="${fb}_${lr}_wheel_joint_motor">
         <hardwareInterface>EffortJointInterface</hardwareInterface>
-        <mechanicalReduction>10</mechanicalReduction>
+        <mechanicalReduction>1</mechanicalReduction>
       </actuator>
     </transmission>
